Commit message: add cmd_vel in car coordinate

File: src/model_description/urdf/LeKiwi_simplified.urdf (robot description, URDF)
Before this commit: robot LeKiwi, 46 links, 45 joints
Links:
- removed link base_link
Joints:
- removed joint base_link_to_chassis

Commit message: change mesh collision geometry to cylinder

File: src/model_description/urdf/LeKiwi_simplified.urdf (robot description, URDF)
Before this commit: robot LeKiwi, 45 links, 44 joints
Links:
- link 4-Omni-Directional-Wheel_Single_Body-v1: geometry collision cylinder length=0.035 radius=0.05; visual mesh filename=package://model_description/meshes/4-Omni-Directional-Wheel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 scale=0.001 0.001 0.001
- link 4-Omni-Directional-Wheel_Single_Body-v1-1: geometry collision cylinder length=0.035 radius=0.05; visual mesh filename=package://model_description/meshes/4-Omni-Directional-Wheel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 scale=0.001 0.001 0.001
- link 4-Omni-Directional-Wheel_Single_Body-v1-2: geometry collision cylinder length=0.035 radius=0.05; visual mesh filename=package://model_description/meshes/4-Omni-Directional-Wheel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 scale=0.001 0.001 0.001

Commit message: configured pid in controllers.yaml and added readme

File: src/model_description/urdf/LeKiwi_simplified.urdf (robot description, URDF)
Before this commit: robot LeKiwi, 45 links, 44 joints
Joints:
- joint ST3215_Servo_Motor-v1-1_Revolute-62: limit (none) -> effort=5.0 velocity=20.0
- joint ST3215_Servo_Motor-v1-2_Revolute-60: limit (none) -> effort=5.0 velocity=20.0
- joint ST3215_Servo_Motor-v1_Revolute-64: limit (none) -> effort=5.0 velocity=20.0

Commit message: update with imu

File: src/model_description/urdf/LeKiwi_simplified.urdf (robot description, URDF)
Before this commit: robot LeKiwi, 45 links, 44 joints
Links:
- added link imu_link; visual box size=0.01 0.01 0.01
Joints:
- added joint imu_joint: type fixed, parent base_plate_layer1-v5, child imu_link, origin xyz=0 0 0.02 rpy=0 0 0

Commit message: add odom frame for rviz

File: src/model_description/urdf/LeKiwi_simplified.urdf (robot description, URDF)
Before this commit: robot LeKiwi, 46 links, 45 joints
Links:
- added link base_link
Joints:
- added joint base_link_to_chassis: type fixed, parent base_link, child base_plate_layer1-v5, origin xyz=0 0 0 rpy=0 0 0

Commit message: ground_truth pub & camera now

File: src/model_description/urdf/LeKiwi_simplified.urdf (robot description, URDF)
Before this commit: robot LeKiwi, 47 links, 46 joints
Links:
- added link camera_link; visual box size=0.005 0.005 0.005
- added link camera_link_optical
Joints:
- added joint camera_link_joint: type fixed, parent Camera-Mount-v8, child camera_link, origin xyz=-0.020 0.035 0.028 rpy=0 0 1.57079632679
- added joint camera_optical_joint: type fixed, parent camera_link, child camera_link_optical, origin xyz=0 0 0 rpy=-1.57079632679 0 -1.57079632679

Commit message: add some content on urdf and plugin

File: src/model_description/urdf/LeKiwi_simplified.urdf (robot description, URDF)
Before this commit: robot LeKiwi, 49 links, 48 joints
Links:
- removed link camera_link
- removed link camera_link_optical
Joints:
- removed joint camera_link_joint
- removed joint camera_optical_joint
